Commit message: bug fix

File: robots/pioneer3at.xacro (robot description, xacro)
@@ -18,5 +18,5 @@
 			<origin xyz="0 0 0.177" rpy="0 0 0"/>
 			<geometry name="pioneer_geom">
-				<mesh filename="package://p3at_tutorial/meshes/p3at_meshes/chassis.stl"/>
+				<mesh filename="package://fcr2017/meshes/p3at_meshes/chassis.stl"/>
 			</geometry>
 			<material name="ChassisRed">
@@ -27,5 +27,5 @@
 			<origin xyz="0 0 0.177" rpy="0 0 0"/>
 				<geometry>
-					<mesh filename="package://p3at_tutorial/meshes/p3at_meshes/chassis.stl"/>
+					<mesh filename="package://fcr2017/meshes/p3at_meshes/chassis.stl"/>
 				</geometry>
 		</collision>
@@ -61,5 +61,5 @@
 			<origin xyz="0 0 0" rpy="0 0 0"/>
 			<geometry name="pioneer_geom">
-				<mesh filename="package://p3at_tutorial/meshes/p3at_meshes/top.stl"/>
+				<mesh filename="package://fcr2017/meshes/p3at_meshes/top.stl"/>
 			</geometry>
 			<material name="TopBlack">
@@ -93,5 +93,5 @@
 			<origin xyz="0 0 0" rpy="0 0 0"/>
 			<geometry name="pioneer_geom">
-				<mesh filename="package://p3at_tutorial/meshes/p3at_meshes/front_sonar.stl"/>
+				<mesh filename="package://fcr2017/meshes/p3at_meshes/front_sonar.stl"/>
 			</geometry>
 			<material name="SonarYellow">
@@ -124,5 +124,5 @@
 			<origin xyz="0 0 0" rpy="0 0 0"/>
 			<geometry name="pioneer_geom">
-				<mesh filename="package://p3at_tutorial/meshes/p3at_meshes/back_sonar.stl"/>
+				<mesh filename="package://fcr2017/meshes/p3at_meshes/back_sonar.stl"/>
 			</geometry>
 			<material name="SonarYellow">
@@ -155,5 +155,5 @@
             <origin xyz="0 0 0" rpy="0 0 0"/>
             <geometry name="pioneer_geom">
-                <mesh filename="package://p3at_tutorial/meshes/p3at_meshes/back_sonar.stl"/>
+                <mesh filename="package://fcr2017/meshes/p3at_meshes/back_sonar.stl"/>
             </geometry>
             <material name="SonarYellow">
@@ -183,5 +183,5 @@
             <origin xyz="0 0 0" rpy="0 0 0"/>
             <geometry name="pioneer_geom">
-                <mesh filename="package://p3at_tutorial/meshes/p3at_meshes/back_sonar.stl"/>
+                <mesh filename="package://fcr2017/meshes/p3at_meshes/back_sonar.stl"/>
             </geometry>
             <material name="SonarYellow">
@@ -213,5 +213,5 @@
 		<origin xyz="0 0 0" rpy="0 0 0"/>
 		<geometry name="pioneer_geom">
-			<mesh filename="package://p3at_tutorial/meshes/p3at_meshes/axle.stl"/>
+			<mesh filename="package://fcr2017/meshes/p3at_meshes/axle.stl"/>
 		</geometry>
 		<material name="AxleGrey">
@@ -244,5 +244,5 @@
 		<origin xyz="0 0 0" rpy="0 0 0"/>
 		<geometry name="pioneer_geom">
-			<mesh filename="package://p3at_tutorial/meshes/p3at_meshes/${suffix}_hubcap.stl"/>
+			<mesh filename="package://fcr2017/meshes/p3at_meshes/${suffix}_hubcap.stl"/>
 		</geometry>
 		<material name="HubcapYellow">
@@ -275,5 +275,5 @@
 		<origin xyz="0 0 0" rpy="0 0 0"/>
 		<geometry name="pioneer_geom">
-			<mesh filename="package://p3at_tutorial/meshes/p3at_meshes/wheel.stl"/>
+			<mesh filename="package://fcr2017/meshes/p3at_meshes/wheel.stl"/>
 		</geometry>
 		<material name="WheelBlack">
@@ -284,5 +284,5 @@
 		<origin xyz="0 0 0" rpy="${-3.1415927/2} 0 0"/>
 		<geometry>
-	    <!--mesh filename="package://p3at_tutorial/meshes/p3at_meshes/wheel.stl"/-->
+	    <!--mesh filename="package://fcr2017/meshes/p3at_meshes/wheel.stl"/-->
 	    <cylinder radius="0.111" length="0.075"/>
 		</geometry>
@@ -312,5 +312,5 @@
 		<origin xyz="0 0 0" rpy="0 0 0"/>
 		<geometry name="pioneer_geom">
-			<mesh filename="package://p3at_tutorial/meshes/p3at_meshes/axle.stl"/>
+			<mesh filename="package://fcr2017/meshes/p3at_meshes/axle.stl"/>
 		</geometry>
 		<material name="AxleGrey">
@@ -321,5 +321,5 @@
 		<origin xyz="0 0 0" rpy="0 0 0"/>
 		<geometry>
-			<mesh filename="package://p3at_tutorial/meshes/p3at_meshes/axle.stl"/>
+			<mesh filename="package://fcr2017/meshes/p3at_meshes/axle.stl"/>
 		</geometry>
 	</collision>
@@ -343,5 +343,5 @@
 		<origin xyz="0 0 0" rpy="0 0 0"/>
 		<geometry name="pioneer_geom">
-			<mesh filename="package://p3at_tutorial/meshes/p3at_meshes/${suffix}_hubcap.stl"/>
+			<mesh filename="package://fcr2017/meshes/p3at_meshes/${suffix}_hubcap.stl"/>
 		</geometry>
 		<material name="HubcapYellow"/>
@@ -350,5 +350,5 @@
 		<origin xyz="0 0 0" rpy="0 0 0"/>
 		<geometry>
-			<mesh filename="package://p3at_tutorial/meshes/p3at_meshes/${suffix}_hubcap.stl"/>
+			<mesh filename="package://fcr2017/meshes/p3at_meshes/${suffix}_hubcap.stl"/>
 		</geometry>
 	</collision>
@@ -372,5 +372,5 @@
 		<origin xyz="0 0 0" rpy="0 0 0"/>
 		<geometry name="pioneer_geom">
-			<mesh filename="package://p3at_tutorial/meshes/p3at_meshes/wheel.stl"/>
+			<mesh filename="package://fcr2017/meshes/p3at_meshes/wheel.stl"/>
 		</geometry>
 		<material name="WheelBlack"/>
@@ -379,5 +379,5 @@
 		<origin xyz="0 0 0" rpy="${-3.1415927/2} 0 0"/>
 		<geometry>
-	    <!--mesh filename="package://p3at_tutorial/meshes/p3at_meshes/wheel.stl"/-->
+	    <!--mesh filename="package://fcr2017/meshes/p3at_meshes/wheel.stl"/-->
 	    <cylinder radius="0.111" length="0.075"/>
 		</geometry>
@@ -451,5 +451,5 @@
       <origin xyz="0 0 0" rpy="0 0 0"/>
       <geometry>
-        <mesh filename="package://p3at_tutorial/meshes/hokuyo1.dae"/>
+        <mesh filename="package://fcr2017/meshes/hokuyo1.dae"/>
       </geometry>
     </visual>
@@ -498,5 +498,5 @@
     <sensor type="ray" name="front_sonar_sensor">
       <pose>0 0 0 0 0 0</pose>
-      <visualize>true</visualize>
+      <visualize>false</visualize>
       <update_rate>25</update_rate>
       <ray>
@@ -537,5 +537,5 @@
     <sensor type="ray" name="back_sonar_sensor">
       <pose>0 0 0 0 0 0</pose>
-      <visualize>true</visualize>
+      <visualize>false</visualize>
       <update_rate>25</update_rate>
       <ray>

Commit message: fix model, add collada files for gazebo 7

File: robots/pioneer3at.xacro (robot description, xacro)
@@ -10,5 +10,5 @@
 		<inertial>
 			<mass value="10.0"/>
-			<origin xyz="0 0 0.177"/>
+			<origin xyz="0 0 0.197"/>
 			<inertia ixx="0.3338" ixy="0.0" ixz="0.0"
 				 iyy="0.4783" iyz="0.0"
@@ -16,7 +16,7 @@
 		</inertial>
 		<visual name="base_visual">
-			<origin xyz="0 0 0.177" rpy="0 0 0"/>
+			<origin xyz="0 0 0.197" rpy="0 0 0"/>
 			<geometry name="pioneer_geom">
-				<mesh filename="package://fcr2017/meshes/p3at_meshes/chassis.stl"/>
+				<mesh filename="package://fcr2017/meshes/p3at_meshes/chassis.dae"/>
 			</geometry>
 			<material name="ChassisRed">
@@ -25,7 +25,7 @@
 		</visual>
 		<collision>
-			<origin xyz="0 0 0.177" rpy="0 0 0"/>
+			<origin xyz="0 0 0.197" rpy="0 0 0"/>
 				<geometry>
-					<mesh filename="package://fcr2017/meshes/p3at_meshes/chassis.stl"/>
+					<mesh filename="package://fcr2017/meshes/p3at_meshes/chassis.dae"/>
 				</geometry>
 		</collision>
@@ -61,5 +61,5 @@
 			<origin xyz="0 0 0" rpy="0 0 0"/>
 			<geometry name="pioneer_geom">
-				<mesh filename="package://fcr2017/meshes/p3at_meshes/top.stl"/>
+				<mesh filename="package://fcr2017/meshes/p3at_meshes/top.dae"/>
 			</geometry>
 			<material name="TopBlack">
@@ -70,5 +70,5 @@
 			<origin xyz="0 0 0" rpy="0 0 0"/>
 			<geometry>
-				<box size="0 0 0"/>
+				<box size="0.01 0.01 0.01"/>
 			</geometry>
 		</collision>
@@ -78,5 +78,5 @@
 	</gazebo>
 	<joint name="base_top_joint" type="fixed">
-		<origin xyz="0.003 0 0.274" rpy="0 0 0"/>
+		<origin xyz="0.040 0 0.274" rpy="0 0 0"/>
 		<parent link="base_link"/>
 		<child link="top_plate"/>
@@ -93,5 +93,5 @@
 			<origin xyz="0 0 0" rpy="0 0 0"/>
 			<geometry name="pioneer_geom">
-				<mesh filename="package://fcr2017/meshes/p3at_meshes/front_sonar.stl"/>
+				<mesh filename="package://fcr2017/meshes/p3at_meshes/front_sonar.dae"/>
 			</geometry>
 			<material name="SonarYellow">
@@ -102,5 +102,5 @@
 			<origin xyz="0 0 0" rpy="0 0 0"/>
 			<geometry>
-				<box size="0 0 0"/>
+				<box size="0.01 0.01 0.01"/>
 			</geometry>
 		</collision>
@@ -124,5 +124,5 @@
 			<origin xyz="0 0 0" rpy="0 0 0"/>
 			<geometry name="pioneer_geom">
-				<mesh filename="package://fcr2017/meshes/p3at_meshes/back_sonar.stl"/>
+				<mesh filename="package://fcr2017/meshes/p3at_meshes/back_sonar.dae"/>
 			</geometry>
 			<material name="SonarYellow">
@@ -133,5 +133,5 @@
 			<origin xyz="0 0 0" rpy="0 0 0"/>
 			<geometry>
-				<box size="0 0 0"/>
+				<box size="0.01 0.01 0.01"/>
 			</geometry>
 		</collision>
@@ -141,5 +141,5 @@
 	</gazebo>
 	<joint name="base_back_joint" type="fixed">
-		<origin xyz="-0.187 0 0.247" rpy="0 0 0"/>
+		<origin xyz="-0.193 0 0.25" rpy="0 0 0"/>
 		<parent link="base_link"/>
 		<child link="back_sonar"/>
@@ -164,5 +164,5 @@
             <origin xyz="0 0 0" rpy="0 0 0"/>
             <geometry>
-                <box size="0 0 0"/>
+                <box size="0.01 0.01 0.01"/>
             </geometry>
         </collision> -->
@@ -192,5 +192,5 @@
             <origin xyz="0 0 0" rpy="0 0 0"/>
             <geometry>
-                <box size="0 0 0"/>
+                <box size="0.01 0.01 0.01"/>
             </geometry>
         </collision> -->
@@ -213,5 +213,5 @@
 		<origin xyz="0 0 0" rpy="0 0 0"/>
 		<geometry name="pioneer_geom">
-			<mesh filename="package://fcr2017/meshes/p3at_meshes/axle.stl"/>
+			<mesh filename="package://fcr2017/meshes/p3at_meshes/axle.dae"/>
 		</geometry>
 		<material name="AxleGrey">
@@ -222,5 +222,5 @@
 		<origin xyz="0 0 0" rpy="0 0 0"/>
 		<geometry>
-			<box size="0 0 0"/>
+			<box size="0.01 0.01 0.01"/>
 		</geometry>
 	</collision>
@@ -244,5 +244,5 @@
 		<origin xyz="0 0 0" rpy="0 0 0"/>
 		<geometry name="pioneer_geom">
-			<mesh filename="package://fcr2017/meshes/p3at_meshes/${suffix}_hubcap.stl"/>
+			<mesh filename="package://fcr2017/meshes/p3at_meshes/${suffix}_hubcap.dae"/>
 		</geometry>
 		<material name="HubcapYellow">
@@ -253,5 +253,5 @@
 		<origin xyz="0 0 0" rpy="0 0 0"/>
 		<geometry>
-			<box size="0 0 0"/>
+			<box size="0.01 0.01 0.01"/>
 		</geometry>
 	</collision>
@@ -261,5 +261,5 @@
 	</gazebo>
 	<joint name="base_front_${suffix}_hub_joint" type="fixed">
-		<origin xyz="0 ${reflect*0.041} 0" rpy="0 0 0"/>
+		<origin xyz="0 ${reflect*0.050} 0" rpy="0 0 0"/>
 		<parent link="p3at_front_${suffix}_axle"/>
 		<child link="p3at_front_${suffix}_hub"/>
@@ -275,5 +275,5 @@
 		<origin xyz="0 0 0" rpy="0 0 0"/>
 		<geometry name="pioneer_geom">
-			<mesh filename="package://fcr2017/meshes/p3at_meshes/wheel.stl"/>
+			<mesh filename="package://fcr2017/meshes/p3at_meshes/wheel.dae"/>
 		</geometry>
 		<material name="WheelBlack">
@@ -312,5 +312,5 @@
 		<origin xyz="0 0 0" rpy="0 0 0"/>
 		<geometry name="pioneer_geom">
-			<mesh filename="package://fcr2017/meshes/p3at_meshes/axle.stl"/>
+			<mesh filename="package://fcr2017/meshes/p3at_meshes/axle.dae"/>
 		</geometry>
 		<material name="AxleGrey">
@@ -321,5 +321,5 @@
 		<origin xyz="0 0 0" rpy="0 0 0"/>
 		<geometry>
-			<mesh filename="package://fcr2017/meshes/p3at_meshes/axle.stl"/>
+			<mesh filename="package://fcr2017/meshes/p3at_meshes/axle.dae"/>
 		</geometry>
 	</collision>
@@ -343,5 +343,5 @@
 		<origin xyz="0 0 0" rpy="0 0 0"/>
 		<geometry name="pioneer_geom">
-			<mesh filename="package://fcr2017/meshes/p3at_meshes/${suffix}_hubcap.stl"/>
+			<mesh filename="package://fcr2017/meshes/p3at_meshes/${suffix}_hubcap.dae"/>
 		</geometry>
 		<material name="HubcapYellow"/>
@@ -350,5 +350,5 @@
 		<origin xyz="0 0 0" rpy="0 0 0"/>
 		<geometry>
-			<mesh filename="package://fcr2017/meshes/p3at_meshes/${suffix}_hubcap.stl"/>
+			<mesh filename="package://fcr2017/meshes/p3at_meshes/${suffix}_hubcap.dae"/>
 		</geometry>
 	</collision>
@@ -358,5 +358,5 @@
 	</gazebo>
 	<joint name="p3at_back_${suffix}_hub_joint" type="fixed">
-		<origin xyz="-0 ${reflect*0.041} 0" rpy="0 0 0"/>
+		<origin xyz="-0 ${reflect*0.050} 0" rpy="0 0 0"/>
 		<parent link="p3at_back_${suffix}_axle"/>
 		<child link="p3at_back_${suffix}_hub"/>
@@ -372,5 +372,5 @@
 		<origin xyz="0 0 0" rpy="0 0 0"/>
 		<geometry name="pioneer_geom">
-			<mesh filename="package://fcr2017/meshes/p3at_meshes/wheel.stl"/>
+			<mesh filename="package://fcr2017/meshes/p3at_meshes/wheel.dae"/>
 		</geometry>
 		<material name="WheelBlack"/>
@@ -399,7 +399,7 @@
     <kp>1000000.0</kp> <!-- kp and kd for rubber -->
     <kd>100.0</kd>
-    <mu1>10.0</mu1>
+    <mu1>1.0</mu1>
     <mu2>1.0</mu2>
-    <fdir1>0 1 0</fdir1> <!-- is this correct? -->
+    <fdir1>1 0 0</fdir1> <!-- is this correct? -->
     <maxVel>1.0</maxVel>
     <minDepth>0.00</minDepth>
@@ -408,7 +408,7 @@
     <kp>1000000.0</kp> <!-- kp and kd for rubber -->
     <kd>100.0</kd>
-    <mu1>10.0</mu1>
+    <mu1>1.0</mu1>
     <mu2>1.0</mu2>
-    <fdir1>0 1 0</fdir1> <!-- is this correct? -->
+    <fdir1>1 0 0</fdir1> <!-- is this correct? -->
     <maxVel>1.0</maxVel>
     <minDepth>0.00</minDepth>
@@ -445,5 +445,5 @@
       <origin xyz="0 0 0" rpy="0 0 0"/>
       <geometry>
-    <box size="0 0 0"/>
+    <box size="0.01 0.01 0.01"/>
       </geometry>
     </collision>
@@ -451,5 +451,5 @@
       <origin xyz="0 0 0" rpy="0 0 0"/>
       <geometry>
-        <mesh filename="package://fcr2017/meshes/hokuyo1.dae"/>
+        <mesh filename="package://fcr2017/meshes/hokuyo.dae"/>
       </geometry>
     </visual>

Commit message: Add PTZ Camera in robot model

File: robots/pioneer3at.xacro (robot description, xacro)
@@ -6,4 +6,5 @@
 name="pioneer3at"
 >
+    <xacro:include filename="$(find fcr2017)/robots/camera.urdf"/>
 <!-- Chassis -->
 	<link name="base_link">
@@ -34,19 +35,9 @@
 		<material value="Gazebo/Red"/>
 	</gazebo>
-<!--link name="odom">
-</link>
-<joint name="odom_base" type="floating">
-		<origin xyz="0 0 0" rpy="0 0 0"/>
-		<parent link="odom"/>
-		<child link="base_link"/>
-	</joint-->
-<!--<link name="map">
-</link-->
-<!--<joint name="map_odom" type="fixed">
-		<origin xyz="0 0 0" rpy="0 0 0"/>
-		<parent link="map"/>
-		<child link="odom"/>
-	</joint>
-	-->
+	<joint name="camera_joint" type="fixed">
+		<origin xyz="0.195 0 0.155" rpy="1.57 0 1.57" />
+		<parent link="base_link" />
+		<child link="pan_link" />
+	</joint>
 <!-- Top -->
 	<link name="top_plate">

Commit message: Add PTZ Camera to the model

File: robots/pioneer3at.xacro (robot description, xacro)
@@ -6,4 +6,5 @@
 name="pioneer3at"
 >
+	<xacro:include filename="$(find fcr2017)/robots/camera.urdf"/>
 <!-- Chassis -->
 	<link name="base_link">
@@ -34,19 +35,9 @@
 		<material value="Gazebo/Red"/>
 	</gazebo>
-<!--link name="odom">
-</link>
-<joint name="odom_base" type="floating">
-		<origin xyz="0 0 0" rpy="0 0 0"/>
-		<parent link="odom"/>
-		<child link="base_link"/>
-	</joint-->
-<!--<link name="map">
-</link-->
-<!--<joint name="map_odom" type="fixed">
-		<origin xyz="0 0 0" rpy="0 0 0"/>
-		<parent link="map"/>
-		<child link="odom"/>
-	</joint>
-	-->
+	<joint name="camera_joint" type="fixed">
+		<origin xyz="0.195 0 0.155" rpy="1.57 0 1.57" />
+		<parent link="base_link"/>
+		<child link="pan_link"/>
+	</joint>
 <!-- Top -->
 	<link name="top_plate">
