Commit message: Joint fix

File: robots/pioneer3at.gazebo.xacro (robot description, xacro)
@@ -10,6 +10,6 @@
     <link name="ptz_camera_optical_gazebo_frame" />
     <joint name="ptz_camera_optical_gazebo_joint" type="fixed">
-      <origin xyz="0.00 0.00 0.055" rpy="-1.57 -1.57 0"/>
-      <parent link="zoom_link" />
+      <origin xyz="0.00 0.00 0.0" rpy="-1.57 -1.57 0"/>
+      <parent link="ptz_camera_optical_frame" />
       <child link="ptz_camera_optical_gazebo_frame"/>
     </joint>

Commit message: Fix joint rotation

File: robots/pioneer3at.gazebo.xacro (robot description, xacro)
@@ -10,5 +10,5 @@
     <link name="ptz_camera_optical_gazebo_frame" />
     <joint name="ptz_camera_optical_gazebo_joint" type="fixed">
-      <origin xyz="0.00 0.00 0.0" rpy="-1.57 -1.57 0"/>
+      <origin xyz="0.00 0.00 0.0" rpy="1.57 -1.57 0"/>
       <parent link="ptz_camera_optical_frame" />
       <child link="ptz_camera_optical_gazebo_frame"/>
