Commit message: Add p controller for ptz camera

File: robots/camera.urdf (robot description, URDF)
Before this commit: robot camera, 3 links, 2 joints
Joints:
- joint pan_joint: limit lower=-1.57 upper=1.57 effort=0 velocity=0 -> lower=-1.57 upper=1.57 effort=1 velocity=1
- joint tilt_joint: limit lower=0 upper=1.57 effort=0 velocity=0 -> lower=0 upper=1.57 effort=1 velocity=1

File: robots/pioneer3at.xacro (robot description, xacro)
@@ -7,6 +7,14 @@
 >
 	<xacro:include filename="$(find fcr2017)/robots/camera.urdf"/>
+<!-- Base Link -->
+	<link name="base_link">
+	</link>
+	<joint name="chassis_joint" type="fixed">
+		<origin xyz="0.0 0 0.0" rpy="0 0 0" />
+		<parent link="base_link"/>
+		<child link="chassis"/>
+	</joint>
 <!-- Chassis -->
-	<link name="base_link">
+	<link name="chassis">
 		<inertial>
 			<mass value="10.0"/>
@@ -32,10 +40,10 @@
 		</collision>
 	</link>
-	<gazebo reference="base_link">
+	<gazebo reference="chassis">
 		<material value="Gazebo/Red"/>
 	</gazebo>
 	<joint name="camera_joint" type="fixed">
 		<origin xyz="0.195 0 0.155" rpy="1.57 0 1.57" />
-		<parent link="base_link"/>
+		<parent link="chassis"/>
 		<child link="pan_link"/>
 	</joint>
@@ -70,5 +78,5 @@
 	<joint name="base_top_joint" type="fixed">
 		<origin xyz="0.040 0 0.274" rpy="0 0 0"/>
-		<parent link="base_link"/>
+		<parent link="chassis"/>
 		<child link="top_plate"/>
 	</joint>
@@ -102,5 +110,5 @@
 	<joint name="base_front_joint" type="fixed">
 		<origin xyz="0.193 0 0.25" rpy="0 0 0"/>
-		<parent link="base_link"/>
+		<parent link="chassis"/>
 		<child link="front_sonar"/>
 	</joint>
@@ -133,5 +141,5 @@
 	<joint name="base_back_joint" type="fixed">
 		<origin xyz="-0.193 0 0.25" rpy="0 0 0"/>
-		<parent link="base_link"/>
+		<parent link="chassis"/>
 		<child link="back_sonar"/>
 	</joint>
@@ -189,5 +197,5 @@
 <joint name="imu_joint" type="fixed">
     <origin xyz="0 0 0" rpy="3.1415 0 0"/>
-    <parent link="base_link"/>
+    <parent link="chassis"/>
     <child link="imu"/>
 </joint>
@@ -222,5 +230,5 @@
 	<joint name="base_front_${suffix}_axle_joint" type="fixed">
 		<origin xyz="0.135 ${reflect*0.156} 0.111" rpy="0 0 0"/>
-		<parent link="base_link"/>
+		<parent link="chassis"/>
 		<child link="p3at_front_${suffix}_axle"/>
 	</joint>
@@ -321,5 +329,5 @@
 	<joint name="p3at_back_${suffix}_axle_joint" type="fixed">
 		<origin xyz="-0.134 ${reflect*0.156} 0.111" rpy="0 0 0"/>
-		<parent link="base_link"/>
+		<parent link="chassis"/>
 		<child link="p3at_back_${suffix}_axle"/>
 	</joint>
@@ -578,4 +586,29 @@
     </plugin>
 </gazebo>
+  <transmission name="pan_trans">
+    <type>transmission_interface/SimpleTransmission</type>
+    <joint name="pan_joint">
+      <hardwareInterface>EffortJointInterface</hardwareInterface>
+    </joint>
+    <actuator name="pan_servo">
+      <hardwareInterface>EffortJointInterface</hardwareInterface>
+      <mechanicalReduction>1</mechanicalReduction>
+    </actuator>
+  </transmission>
+  <transmission name="tilt_trans">
+    <type>transmission_interface/SimpleTransmission</type>
+    <joint name="tilt_joint">
+      <hardwareInterface>EffortJointInterface</hardwareInterface>
+    </joint>
+    <actuator name="tilt_servo">
+      <hardwareInterface>EffortJointInterface</hardwareInterface>
+      <mechanicalReduction>1</mechanicalReduction>
+    </actuator>
+  </transmission>
+<gazebo>
+  <plugin name="gazebo_ros_control" filename="libgazebo_ros_control.so">
+    <robotNamespace>/</robotNamespace>
+  </plugin>
+</gazebo>
 </xacro:macro>
 <xacro:p3at_front suffix="left" reflect="1"/>

Commit message: Add camera plugin to the PTZ Camera in Gazebo

File: robots/camera.urdf (robot description, URDF)
Before this commit: robot camera, 3 links, 2 joints
Joints:
- joint pan_joint: limit lower=-1.57 upper=1.57 effort=1 velocity=1 -> lower=-1.5707963267948966 upper=1.5707963267948966 effort=1 velocity=1.5707963267948966
- joint tilt_joint: limit lower=0 upper=1.57 effort=1 velocity=1 -> lower=-0.5235987755982988 upper=1.5707963267948966 effort=1 velocity=1.2217304763960306

File: robots/pioneer3at.xacro (robot description, xacro)
@@ -462,5 +462,5 @@
     <sensor type="ray" name="head_hokuyo_sensor">
       <pose>0 0 0 0 0 0</pose>
-      <visualize>true</visualize>
+      <visualize>false</visualize>
       <update_rate>40</update_rate>
       <ray>
@@ -606,9 +606,16 @@
     </actuator>
   </transmission>
-<gazebo>
-  <plugin name="gazebo_ros_control" filename="libgazebo_ros_control.so">
-    <robotNamespace>/</robotNamespace>
-  </plugin>
-</gazebo>
+  <gazebo>
+    <plugin name="gazebo_ros_control" filename="libgazebo_ros_control.so">
+      <robotNamespace>/</robotNamespace>
+    </plugin>
+  </gazebo>
+<!-- Camera Frame for ROS -->
+    <link name="ptz_camera_optical_frame" />
+    <joint name="ptz_camera_optical_joint" type="fixed">
+      <origin xyz="0.00 0.00 0.055" rpy="0 0 3.14"/>
+      <parent link="zoom_link" />
+      <child link="ptz_camera_optical_frame"/>
+    </joint>
 </xacro:macro>
 <xacro:p3at_front suffix="left" reflect="1"/>

Commit message: Add PTZ camera to the model, p control for pan tilt

File: robots/camera.urdf (robot description, URDF)
Before this commit: robot camera, 3 links, 2 joints
Links:
- link pan_link: geometry collision mesh filename=package://fcr2017/meshes/ptz_canon_camera/pan_link.stl; visual mesh filename=package://fcr2017/meshes/ptz_canon_camera/pan_link.stl
- link tilt_link: geometry collision mesh filename=package://fcr2017/meshes/ptz_canon_camera/tilt_link.stl; visual mesh filename=package://fcr2017/meshes/ptz_canon_camera/tilt_link.stl
- link zoom_link: geometry collision mesh filename=package://fcr2017/meshes/ptz_canon_camera/zoom_link.stl; visual mesh filename=package://fcr2017/meshes/ptz_canon_camera/zoom_link.stl
Joints:
- joint pan_joint: limit lower=-1.57 upper=1.57 effort=0 velocity=0 -> lower=-1.5707963267948966 upper=1.5707963267948966 effort=1 velocity=1.5707963267948966
- joint tilt_joint: limit lower=0 upper=1.57 effort=0 velocity=0 -> lower=-0.5235987755982988 upper=1.5707963267948966 effort=1 velocity=1.2217304763960306

File: robots/pioneer3at.xacro (robot description, xacro)
@@ -578,4 +578,36 @@
     </plugin>
 </gazebo>
+  <transmission name="pan_trans">
+    <type>transmission_interface/SimpleTransmission</type>
+    <joint name="pan_joint">
+      <hardwareInterface>EffortJointInterface</hardwareInterface>
+    </joint>
+    <actuator name="pan_servo">
+      <hardwareInterface>EffortJointInterface</hardwareInterface>
+      <mechanicalReduction>1</mechanicalReduction>
+    </actuator>
+  </transmission>
+  <transmission name="tilt_trans">
+    <type>transmission_interface/SimpleTransmission</type>
+    <joint name="tilt_joint">
+      <hardwareInterface>EffortJointInterface</hardwareInterface>
+    </joint>
+    <actuator name="tilt_servo">
+      <hardwareInterface>EffortJointInterface</hardwareInterface>
+      <mechanicalReduction>1</mechanicalReduction>
+    </actuator>
+  </transmission>
+  <gazebo>
+    <plugin name="gazebo_ros_control" filename="libgazebo_ros_control.so">
+      <robotNamespace>/</robotNamespace>
+    </plugin>
+  </gazebo>
+<!-- Camera Frame for ROS -->
+    <link name="ptz_camera_optical_frame" />
+    <joint name="ptz_camera_optical_joint" type="fixed">
+      <origin xyz="0.00 0.00 0.055" rpy="0 0 3.14"/>
+      <parent link="zoom_link" />
+      <child link="ptz_camera_optical_frame"/>
+    </joint>
 </xacro:macro>
 <xacro:p3at_front suffix="left" reflect="1"/>

Commit message: Fixing camera

File: robots/camera.urdf (robot description, URDF)
Before this commit: robot camera, 3 links, 2 joints
Joints:
- joint pan_joint: origin xyz=0 0 0.0127 rpy=-4.5919E-16 -1.7382E-16 -3.136 -> xyz=0 0 0.0127 rpy=-4.5919E-16 -1.7382E-16 1.57; type revolute -> fixed
- joint tilt_joint: type revolute -> fixed
